Commit message: Fix zed2i mesh path

File: ws_moveit/src/group1/config/final_setup.urdf (robot description, URDF)
Before this commit: robot m_robot, 28 links, 27 joints
Links:
- link zed2i_camera_center: geometry collision mesh filename=package://iiwa_description/meshes/zed2i.stl; visual mesh filename=package://iiwa_description/meshes/zed2i.stl

Commit message: Fix zed2i mesh path

File: ws_moveit/src/group1/config/final_setup.urdf (robot description, URDF)
Before this commit: robot m_robot, 28 links, 27 joints
Links:
- link zed2i_camera_center: geometry collision mesh filename=package://iiwa_description/meshes/zed2i/zed2i.stl; visual mesh filename=package://iiwa_description/meshes/zed2i/zed2i.stl

Commit message: Fix: Gazebo
Now you can run roslaunch group1 demo_gazebo.launch to start a Gazebo simulation and launch Rviz.

File: ws_moveit/src/group1/config/final_setup.urdf (robot description, URDF)
Before this commit: robot m_robot, 28 links, 27 joints
Links:
- link m_robot_support_structure: mass 0.1 -> 0.001
